File: SerialServerBoard/security.kicad_sch (KiCad schematic)
At the start: 0 parts

Commit message: Add ATECC
Parts:
- added C13: TBD, Capacitor_SMD:C_0603_1608Metric, symbol Device:C_Small
- added U4: ATECC608B-MAHDA, Package_DFN_QFN:DFN-8-1EP_3x2mm_P0.5mm_EP1.3x1.5mm, symbol Security:ATECC608B-MAHDA
Connections:
- new net +3V3_SW: C13.1, U4.8 (VCC)
- new net GND: C13.2, U4.4 (GND), U4.9 (EP)
- new net I2C_SCL: U4.6 (SCL)
- new net I2C_SDA: U4.5 (SDA)
