File: SerialServerBoard/SerialServerBoard.kicad_sch (KiCad schematic)
At the start: 24 parts, among them J1 3v3, J2 3v3_SW, J3 1v8, J4 1v35, J5 VCORE, SW1 RST, SW2 BOOT

Commit message: Add ATECC
Parts:
- added J9: I2C, Connector_PinHeader_1.27mm:PinHeader_1x04_P1.27mm_Vertical, symbol Connector:Conn_01x04_Pin
Connections:
- net +3V3_SW: now also J9.1 (Pin_1)
- net GND: now also J9.2 (Pin_2)
- new net I2C_SCL: J9.4 (Pin_4)
- new net I2C_SDA: J9.3 (Pin_3)

Commit message: Add micro-SD card slot
Parts:
- added R38, R39: 4k7, Resistor_SMD:R_0603_1608Metric, symbol Device:R_Small
Connections:
- net +3V3_SW: now also R38.1, R39.1
- net I2C_SCL: now also R38.2
- net I2C_SDA: now also R39.2
Other:
- note added: "TODO: Determine more optimal values"
