File: SerialServerBoard/wifi.kicad_sch (KiCad schematic)
At the start: 0 parts

Commit message: Add ESP32-C3 footprint
Parts:
- added FB3: FerriteBead_Small, symbol Device:FerriteBead_Small
- added J10: Conn_ARM_JTAG_SWD_10, Connector_PinSocket_1.27mm:PinSocket_2x05_P1.27mm_Vertical, symbol Connector:Conn_ARM_JTAG_SWD_10
- added J8: ESP UART, Connector_PinSocket_1.27mm:PinSocket_1x04_P1.27mm_Vertical, symbol Connector:Conn_01x04_Pin
- added U3: ESP32-C3, Footprints:ESP32-C3, symbol Symbols:ESP32-C3
Connections:
- new net: J10.8 (NC/TDI), U3.10 (MTDI)
- new net: J10.4 (SWCLK/TCK), U3.12 (MTCK)
- new net: J10.6 (SWO/TDO), U3.13 (MTDO)
- new net: J8.3 (Pin_3), U3.27 (U0RXD)
- new net: J8.4 (Pin_4), U3.28 (U0TXD)
- new net: J10.2 (SWDIO/TMS), U3.9 (MTMS)
- new net +3V3_SW: FB3.1
- new net 3V3_ESP32: FB3.2, J10.1 (VTref), J8.1 (Pin_1), U3.11 (VDD3P3_RTC), U3.17 (VDD3P3_CPU), U3.18 (VDD_SPI), U3.2 (VDD3P3), U3.3 (VDD3P3), U3.31 (VDDA), U3.32 (VDDA)
- new net GND: J10.3 (GND), J10.5 (GND), J10.9 (GNDDetect), J8.2 (Pin_2)
Other:
- note added: "TODO: Check details on power supply - Should VDDA or any other rails have a specific decoupling? - Should VDDA and VDD_SPI be at 3v3?"

Commit message: Add ATECC
Parts:
- FB3: footprint (none) -> Inductor_SMD:L_0603_1608Metric
Changed lines of the file:
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@@
 			)
 		)
-		(property "Footprint" ""
+		(property "Footprint" "Inductor_SMD:L_0603_1608Metric"
 			(at 186.182 38.1 90)
 			(effects

Commit message: Add micro-SD card slot
Parts:
- added R40: 4k7, Resistor_SMD:R_0402_1005Metric, symbol Device:R_Small
Connections:
- net +3V3_SW: now also R40.1
- net at U3.6 (GPIO2): now also R40.2
Other:
- note added: "NOTE: Must use a variant of ESP32-C3 with internal flash"
Changed lines of the file:
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@@
+	(wire
+		(pts
+			(xy 125.73 35.56) (xy 125.73 38.1)
+		)
+		(stroke
+			(width 0)
+			(type default)
+		)
+	)
 	(wire
 		(pts
@@
 	(wire
 		(pts
+			(xy 125.73 43.18) (xy 125.73 46.99)
+		)
+		(stroke
+			(width 0)
+			(type default)
+		)
+	)
+	(wire
+		(pts
+			(xy 125.73 46.99) (xy 130.81 46.99)
+		)
+		(stroke
+			(width 0)
+			(type default)
+		)
+	)
+	(wire
+		(pts
 			(xy 121.92 111.76) (xy 121.92 95.25)
 		)
@@
 			(width 0)
 			(type default)
+		)
+	)
+	(text "NOTE: Must use a variant of ESP32-C3 with internal flash"
+		(exclude_from_sim no)
+		(at 102.616 64.516 0)
+		(effects
+			(font
+				(size 1.27 1.27)
+			)
 		)
 	)
@@
 			)
 			(justify right bottom)
+		)
+	)
+	(symbol
+		(lib_id "Device:R_Small")
+		(at 125.73 40.64 0)
+		(unit 1)
+		(exclude_from_sim no)
+		(in_bom yes)
+		(on_board yes)
+		(dnp no)
+		(fields_autoplaced yes)
+		(property "Reference" "R40"
+			(at 128.27 39.37 0)
+			(effects
+				(font
+					(size 1.27 1.27)
+				)
+				(justify left)
+			)
+		)
+		(property "Value" "4k7"
+			(at 128.27 41.91 0)
+			(effects
+				(font
+					(size 1.27 1.27)
+				)
+				(justify left)
+			)
+		)
+		(property "Footprint" "Resistor_SMD:R_0402_1005Metric"
+			(at 125.73 40.64 0)
+			(effects
+				(font
+					(size 1.27 1.27)
+				)
+				(hide yes)
+			)
+		)
+		(property "Datasheet" "~"
+			(at 125.73 40.64 0)
+			(effects
+				(font
+					(size 1.27 1.27)
+				)
+				(hide yes)
+			)
+		)
+		(property "Description" ""
+			(at 125.73 40.64 0)
+			(effects
+				(font
+					(size 1.27 1.27)
+				)
+				(hide yes)
+			)
+		)
+		(pin "1"
+		)
+		(pin "2"
+		)
+		(instances
+			(project "SerialServerBoard"
+				(path "/fff4edd7-7765-4881-b8c8-325c8be7c8ba/d4043790-84bf-4077-974b-7325bae32458"
+					(reference "R40")
+					(unit 1)
+				)
+			)
 		)
 	)
@@
 					(unit 1)
 				)
+			)
+		)
+	)
+	(symbol
+		(lib_id "Symbols:+3V3_SW")
+		(at 125.73 35.56 0)
+		(unit 1)
+		(exclude_from_sim no)
+		(in_bom yes)
+		(on_board yes)
+		(dnp no)
+		(fields_autoplaced yes)
+		(property "Reference" "#PWR066"
+			(at 125.73 39.37 0)
+			(effects
+				(font
+					(size 1.27 1.27)
+				)
+				(hide yes)
+			)
+		)
+		(property "Value" "+3V3_SW"
+			(at 125.73 30.48 0)
+			(effects
+				(font
+					(size 1.27 1.27)
+				)
+			)
+		)
+		(property "Footprint" ""
+			(at 125.73 35.56 0)
+			(effects
+				(font
+					(size 1.27 1.27)
+				)
+				(hide yes)
+			)
+		)
+		(property "Datasheet" ""
+			(at 125.73 35.56 0)
+			(effects
+				(font
+					(size 1.27 1.27)
+				)
+				(hide yes)
+			)
+		)
+		(property "Description" "Power symbol creates a global label with name \"+3V3_SW\""
+			(at 125.73 35.56 0)
+			(effects
+				(font
+					(size 1.27 1.27)
+				)
+				(hide yes)
+			)
+		)
+		(pin "1"
+		)
+		(instances
+			(project "SerialServerBoard"
+				(path "/fff4edd7-7765-4881-b8c8-325c8be7c8ba/d4043790-84bf-4077-974b-7325bae32458"
+					(reference "#PWR066")
+					(unit 1)
+				)
